Commit message: file structure update

File: src/robot_arm_description/urdf/Robot_Arm.urdf (robot description, URDF)
Before this commit: robot robot_arm, 8 links, 7 joints
Links:
- removed link end_effector
- removed link left_finger
- removed link link1
- removed link link2
- removed link link3
- removed link link4
- removed link right_finger
- added link End-Effector, mass 0.0577947757867498; collision mesh filename=package://Robot_Arm/meshes/End-Effector.STL; visual mesh filename=package://Robot_Arm/meshes/End-Effector.STL
- added link GripL, mass 0.0184570467495853; collision mesh filename=package://Robot_Arm/meshes/GripL.STL; visual mesh filename=package://Robot_Arm/meshes/GripL.STL
- added link GripR, mass 0.0184570467495853; collision mesh filename=package://Robot_Arm/meshes/GripR.STL; visual mesh filename=package://Robot_Arm/meshes/GripR.STL
- added link Link1, mass 0.207180993005197; collision mesh filename=package://Robot_Arm/meshes/Link1.STL; visual mesh filename=package://Robot_Arm/meshes/Link1.STL
- added link Link2, mass 0.0150579864214192; collision mesh filename=package://Robot_Arm/meshes/Link2.STL; visual mesh filename=package://Robot_Arm/meshes/Link2.STL
- added link Link3, mass 0.0411732267600477; collision mesh filename=package://Robot_Arm/meshes/Link3.STL; visual mesh filename=package://Robot_Arm/meshes/Link3.STL
- added link Link4, mass 0.0316676572660873; collision mesh filename=package://Robot_Arm/meshes/Link4.STL; visual mesh filename=package://Robot_Arm/meshes/Link4.STL
- link base_link: mass 0.072556 -> 0.0725564097125622; geometry collision mesh filename=package://Robot_Arm/meshes/base_link.STL; visual mesh filename=package://Robot_Arm/meshes/base_link.STL
Joints:
- removed joint end-joint
- removed joint grip_joint1
- removed joint grip_joint2
- removed joint joint1
- removed joint joint2
- removed joint joint3
- removed joint joint4
- added joint End-Joint: type fixed, parent Link4, child End-Effector, origin xyz=-0.05286 0.019218 -0.029276 rpy=1.5708 0 -3.1416, axis 0 0 0
- added joint Grip_Joint1: type prismatic, parent Link4, child GripL, origin xyz=-0.06744 0.036228 0.0065437 rpy=1.5708 0 3.1416, axis 0 1 0, limit lower=0 upper=0 effort=0 velocity=0
- added joint Grip_Joint2: type prismatic, parent Link4, child GripR, origin xyz=-0.06744 0.036138 -0.065096 rpy=1.5708 0 -3.1416, axis 0 1 0, limit lower=0 upper=0 effort=0 velocity=0
- added joint Joint1: type revolute, parent base_link, child Link1, origin xyz=0 0 0.09255 rpy=0 0 0, axis 0 0 1, limit lower=0 upper=3.1416 effort=0 velocity=0
- added joint Joint2: type revolute, parent Link1, child Link2, origin xyz=0.0108 -0.03605 0.019 rpy=1.5708 0 0, axis 0 0 1, limit lower=0 upper=3.1416 effort=0 velocity=0
- added joint Joint3: type revolute, parent Link2, child Link3, origin xyz=0.103 0 -0.053 rpy=0 0 -1.5708, axis 0 0 1, limit lower=0 upper=3.1416 effort=0 velocity=0
- added joint Joint4: type revolute, parent Link3, child Link4, origin xyz=0.0978 0.0015 -0.00095 rpy=3.1416 0 -1.5708, axis 0 0 1, limit lower=0 upper=3.1416 effort=0 velocity=0
