Commit message: error fix in robot mesh

File: src/robot_arm_description/robot_arm/urdf/robot_arm.urdf (robot description, URDF)
Before this commit: robot Robot_Arm, 8 links, 7 joints
Links:
- removed link End-Effector
- removed link GripL
- removed link GripR
- removed link Link1
- removed link Link2
- removed link Link3
- removed link Link4
- added link end_effector, mass 0.057795; collision mesh filename=package://robot_arm/meshes/end_effector.STL; visual mesh filename=package://robot_arm/meshes/end_effector.STL
- added link left_finger, mass 0.018457; collision mesh filename=package://robot_arm/meshes/left_finger.STL; visual mesh filename=package://robot_arm/meshes/left_finger.STL
- added link link1, mass 0.20718; collision mesh filename=package://robot_arm/meshes/link1.STL; visual mesh filename=package://robot_arm/meshes/link1.STL
- added link link2, mass 0.015058; collision mesh filename=package://robot_arm/meshes/link2.STL; visual mesh filename=package://robot_arm/meshes/link2.STL
- added link link3, mass 0.041173; collision mesh filename=package://robot_arm/meshes/link3.STL; visual mesh filename=package://robot_arm/meshes/link3.STL
- added link link4, mass 0.031668; collision mesh filename=package://robot_arm/meshes/link4.STL; visual mesh filename=package://robot_arm/meshes/link4.STL
- added link right_finger, mass 0.018457; collision mesh filename=package://robot_arm/meshes/right_finger.STL; visual mesh filename=package://robot_arm/meshes/right_finger.STL
- link base_link: mass 0.0725564097125622 -> 0.072556; geometry collision mesh filename=package://robot_arm/meshes/base_link.STL; visual mesh filename=package://robot_arm/meshes/base_link.STL
Joints:
- removed joint End-Joint
- removed joint Grip_Joint1
- removed joint Grip_Joint2
- removed joint Joint1
- removed joint Joint2
- removed joint Joint3
- removed joint Joint4
- added joint end-joint: type fixed, parent link4, child end_effector, origin xyz=-0.05286 0.019218 -0.029276 rpy=1.5708 0 -3.1416, axis 0 0 0
- added joint grip_joint1: type prismatic, parent link4, child left_finger, origin xyz=-0.06744 0.036228 0.0065437 rpy=1.5708 0 3.1416, axis 0 -1 0, limit lower=0 upper=0 effort=0 velocity=0
- added joint grip_joint2: type prismatic, parent link4, child right_finger, origin xyz=-0.06744 0.036138 -0.065096 rpy=1.5708 0 3.1416, axis 0 -1 0, limit lower=0 upper=0 effort=0 velocity=0
- added joint joint1: type revolute, parent base_link, child link1, origin xyz=0 0 0.09255 rpy=0 0 0, axis 0 0 1, limit lower=0 upper=3.1416 effort=0 velocity=0
- added joint joint2: type revolute, parent link1, child link2, origin xyz=0.0108 -0.03605 0.019 rpy=1.5708 0 0, axis 0 0 1, limit lower=0 upper=3.1416 effort=0 velocity=0
- added joint joint3: type revolute, parent link2, child link3, origin xyz=0.103 0 -0.053 rpy=0 0 -1.5708, axis 0 0 1, limit lower=0 upper=3.1416 effort=0 velocity=0
- added joint joint4: type revolute, parent link3, child link4, origin xyz=0.0978 0.0015 -0.00095 rpy=3.1416 0 -1.5708, axis 0 0 1, limit lower=0 upper=3.1416 effort=0 velocity=0
